File: hw/lp/MSP-EXP430F5529LP.sch (EAGLE design)
At the start: 27 parts, among them J10 PWR, J3 PWR, Q2 32.768kHz, Q4 CSTCR4M00G15L99, U6 MSP430F5529IPNR

Commit message: adding usb power need ldos
Parts:
- removed C16: 220n, rcl:C-EUC0402
- removed C20, C21, C402: 100n, rcl:C-EUC0402
- removed C403: 4u7, rcl:CPOL-EUA/3216-18R
- removed J10, J3: PWR, pinhead:PINHD-1X3
- removed J401: (no value), usb_con-update:USB_MICRO_FLIPPED
- removed R401: 33R, rcl:R-EU_R0402
- added C1, C3, C4: 100n, rcl:C-EUC0402
- added C2: 4u7, rcl:CPOL-EUA/3216-18R
- added J1: (no value), usb_con-update:USB_MICRO_FLIPPED
- added J2, J4: PWR, pinhead:PINHD-1X3
- added JP1: JTAG, con-lstb:MA07-2
- added R1: 33R, rcl:R-EU_R0402
- added R2: 330R, rcl:R-EU_R0402
Connections:
- removed net EZFET_VBUS: C402.1, C403.+, J401.VBUS
- removed net N$10: J401.SHIELD1, R401.1
- removed net N$11: U$2.P13
- removed net N$12: J401.D+
- removed net N$13: J401.D-
- removed net N$14: U$2.P12
- removed net N$15: U$2.P11
- removed net N$16: U$2.P10
- removed net N$17: U$2.P9
- removed net N$18: U$2.P8
- removed net N$19: U$2.P7
- removed net N$2: U$2.P2
- removed net N$20: U$2.P6
- removed net N$21: U$2.P5
- removed net N$22: U$2.P4
- removed net N$23: U$2.P3
- removed net N$24: U$2.P21
- removed net N$25: U$2.P22
- removed net N$26: U$2.P23
- removed net N$27: U$2.P24
- removed net N$28: U$2.P25
- removed net N$29: U$2.P26
- removed net N$3: U$2.P18
- removed net N$4: U$2.P20
- removed net N$5: U$2.P17
- removed net N$6: U$2.P16
- removed net N$7: U$2.P15
- removed net N$8: U$2.P14
- removed net TARGET_VUSB: C16.1, U6.66
- new net DM: J1.D-, U6.64
- new net DP: J1.D+, U6.62
- new net N$39: J1.SHIELD1, R1.1
- new net SBWVCC: JP1.2
- new net VUSB: C1.1, C2.+, J1.VBUS, U6.66
- net +3V3: now also C3.1, J2.3; no longer C20.1, J10.3
- net +5V: now also C4.1, J4.3; no longer C21.1, J3.3
- net GND: now also C1.2, C2.-, C3.2, C4.2, J1.GND, J2.1, J2.2, J4.1, J4.2, JP1.9, R1.2; no longer C16.2, C20.2, C21.2, C402.2, C403.-, J10.1, J10.2, J3.1, J3.2, J401.GND, R401.2
- net N$1: now also JP1.7, R2.2; no longer U$2.P1
- net P1.0: now also U$2.P1
- net P1.1: now also U$2.P3
- net P1.2: now also U$2.P5
- net P1.3: now also U$2.P7
- net P1.4: now also U$2.P2
- net P1.5: now also U$2.P4
- net P1.6: now also U$2.P6
- net P1.7: now also U$2.P8
- net P2.0: now also U$2.P9
- net P2.1: now also U$2.P10
- net P2.2: now also U$2.P11
- net P2.3: now also U$2.P12
- net P2.4: now also U$2.P13
- net P2.5: now also U$2.P14
- net P2.6: now also U$2.P15
- net P2.7: now also U$2.P16
- net P3.0: now also U$2.P17
- net P3.1: now also U$2.P18
- net P3.2: now also U$2.P20
- net P3.3: now also U$2.P21
- net P3.4: now also U$2.P22
- net P3.5: now also U$2.P23
- net P3.6: now also U$2.P24
- net P3.7: now also U$2.P25
- net P4.0: now also U$2.P26
- net RST/SBWTDIO: now also JP1.1
- net TEST/SBWTCK: now also JP1.8, R2.1
Other:
- note removed: "1.5"
- note removed: "Connections"
- note removed: "Design Notes:"
- note removed: "Free IO pins: 4.6, 5.0, 5.1, 5.6, 5.7, 7.1, 7.2, 7.3, 7.5, 7.6, 7.7, 8.0, PJ.x (4)"
- note removed: "Main MSP430F5529 w Power, Clock and USB"
- note removed: "Remove R28 and inject AVCC directly if needed"
- note removed: "USB Hub and Power"
